Commit message: Add keyboard teleop hx5_d20 left&right

File: robotis_hand_description/urdf/hx5_d20_rev2/hx5_d20_left.urdf.xacro (robot description, xacro)
@@ -71,5 +71,5 @@
          <origin xyz="0.039 0.0 0.0" rpy="0 0 0" />
          <axis xyz="0 0 1" />
-         <limit velocity="4.8" effort="1000" lower="0.0" upper="3.14" />
+         <limit velocity="4.8" effort="1000" lower="-0.5" upper="3.5" />
          <dynamics damping="0.05" />
       </joint>
@@ -106,5 +106,5 @@
          <origin xyz="0.0 -0.028 0.0" rpy="0 0 0" />
          <axis xyz="1 0 0" />
-         <limit velocity="4.8" effort="1000" lower="-1.57" upper="0.0" />
+         <limit velocity="4.8" effort="1000" lower="-1.57" upper="0.5" />
          <dynamics damping="0.05" />
       </joint>
@@ -141,5 +141,5 @@
          <origin xyz="0.0 -0.0355 0.0" rpy="0 0 0" />
          <axis xyz="1 0 0" />
-         <limit velocity="4.8" effort="1000" lower="-1.57" upper="0.0" />
+         <limit velocity="4.8" effort="1000" lower="-1.57" upper="0.5" />
          <dynamics damping="0.05" />
       </joint>

File: robotis_hand_description/urdf/hx5_d20_rev2/hx5_d20_right.urdf.xacro (robot description, xacro)
@@ -71,5 +71,5 @@
          <origin xyz="0.039 0.0 0.0" rpy="0 0 0" />
          <axis xyz="0 0 1" />
-         <limit velocity="4.8" effort="1000" lower="-3.14" upper="0.0" />
+         <limit velocity="4.8" effort="1000" lower="-3.5" upper="0.5" />
          <dynamics damping="0.05" />
       </joint>
@@ -106,5 +106,5 @@
          <origin xyz="0.0 0.028 0.0" rpy="0 0 0" />
          <axis xyz="1 0 0" />
-         <limit velocity="4.8" effort="1000" lower="0.0" upper="1.57" />
+         <limit velocity="4.8" effort="1000" lower="-0.5" upper="1.57" />
          <dynamics damping="0.05" />
       </joint>
@@ -141,5 +141,5 @@
          <origin xyz="0.0 0.0355 0.0" rpy="0 0 0" />
          <axis xyz="1 0 0" />
-         <limit velocity="4.8" effort="1000" lower="0.0" upper="1.57" />
+         <limit velocity="4.8" effort="1000" lower="-0.5" upper="1.57" />
          <dynamics damping="0.05" />
       </joint>
