Commit message: Add IK for X_bios

File: robotis_hand_description/urdf/hx5_d20_rev2/hx5_d20_right.urdf.xacro (robot description, xacro)
@@ -193,5 +193,5 @@
          <origin xyz="-0.0015 0.03608 0.10275" rpy="0 0 0" />
          <axis xyz="1 0 0" />
-         <limit velocity="4.8" effort="1000" lower="-0.6" upper="0.6" />
+         <limit velocity="4.8" effort="1000" lower="-1.5" upper="0.6" />
          <dynamics damping="0.05" />
       </joint>
@@ -664,5 +664,5 @@
          <origin xyz="-0.0015 -0.04492 0.08575" rpy="0 0 0" />
          <axis xyz="1 0 0" />
-         <limit velocity="4.8" effort="1000" lower="-0.6" upper="0.6" />
+         <limit velocity="4.8" effort="1000" lower="-0.6" upper="1.5" />
          <dynamics damping="0.05" />
       </joint>

Commit message: Add unused finger logic

File: robotis_hand_description/urdf/hx5_d20_rev2/hx5_d20_right.urdf.xacro (robot description, xacro)
@@ -193,5 +193,5 @@
          <origin xyz="-0.0015 0.03608 0.10275" rpy="0 0 0" />
          <axis xyz="1 0 0" />
-         <limit velocity="4.8" effort="1000" lower="-1.5" upper="0.6" />
+         <limit velocity="4.8" effort="1000" lower="-0.6" upper="0.6" />
          <dynamics damping="0.05" />
       </joint>
@@ -664,5 +664,5 @@
          <origin xyz="-0.0015 -0.04492 0.08575" rpy="0 0 0" />
          <axis xyz="1 0 0" />
-         <limit velocity="4.8" effort="1000" lower="-0.6" upper="1.5" />
+         <limit velocity="4.8" effort="1000" lower="-0.6" upper="0.6" />
          <dynamics damping="0.05" />
       </joint>
